Commit message: Test for self-collision

File: rrbot_description/urdf/rrbot.xacro (robot description, xacro)
@@ -79,5 +79,5 @@
     <parent link="link2"/>
     <child link="link3"/>
-    <origin xyz="0 ${width} ${height2 - axel_offset*2}" rpy="0 0 0"/>
+    <origin xyz="0 -${width} ${height2 - axel_offset*2}" rpy="0 0 0"/>
     <axis xyz="0 1 0"/>
     <dynamics damping="0.7"/>
